File: PCB/winter.kicad_pcb (KiCad board)
At the start: 2 copper layers, 319.8 x 101.2 mm, 142 parts, among them SW1 SW_Push, SW10 SW_Push, SW11 SW_Push, SW12 SW_Push, SW13 SW_Push, SW14 SW_Push, SW15 SW_Push, SW16 SW_Push, SW17 SW_Push, SW18 SW_Push, SW19 SW_Push, SW2 SW_Push, SW20 SW_Push, SW21 SW_Push, SW22 SW_Push, SW23 SW_Push, SW24 SW_Push, SW25 SW_Push, SW26 SW_Push, SW27 SW_Push, SW28 SW_Push, SW29 SW_Push, SW3 SW_Push, SW30 SW_Push, SW31 SW_Push, SW32 SW_Push, SW33 SW_Push, SW34 SW_Push, SW35 SW_Push, SW36 SW_Push, SW37 SW_Push, SW38 SW_Push, SW39 SW_Push, SW4 SW_Push, SW40 SW_Push, SW41 SW_Push, SW42 SW_Push, SW43 SW_Push, SW44 SW_Push, SW45 SW_Push, SW46 SW_Push, SW47 SW_Push, SW48 SW_Push, SW49 SW_Push, SW5 SW_Push, SW50 SW_Push, SW51 SW_Push, SW52 SW_Push, SW53 SW_Push, SW54 SW_Push, SW55 SW_Push, SW56 SW_Push, SW57 SW_Push, SW58 SW_Push, SW59 SW_Push, SW6 SW_Push, SW60 SW_Push, SW61 SW_Push, SW62 SW_Push, SW63 SW_Push, SW64 SW_Push, SW65 SW_Push, SW7 SW_Push, SW8 SW_Push, SW9 SW_Push, U1 RP2040-ZERO

Commit message: changed mcu and added screen and knob
Parts:
- removed U1: RP2040-ZERO, Winter60_RP2040:MODULE_RP2040-ZERO_Clean
- added A1: RaspberryPi_Pico, Module:RaspberryPi_Pico_Common_Unspecified, F.Cu at (290.0, 14.0)
- added H7: MountingHole_2.7mm_M2.5_Clean, Winter60_Mounting:MountingHole_2.7mm_M2.5_Clean, F.Cu at (275.0, 28.5)
- added H8: MountingHole_2.7mm_M2.5_Clean, Winter60_Mounting:MountingHole_2.7mm_M2.5_Clean, F.Cu at (275.0, 66.6)
- added J1: Conn_01x04, Connector_PinHeader_2.54mm:PinHeader_1x04_P2.54mm_Vertical, F.Cu at (290.0, 75.0)
- added R1: 10k, Resistor_SMD:R_0805_2012Metric, F.Cu at (280.0, 48.0)
- added R2: 4.7k, Resistor_SMD:R_0805_2012Metric, F.Cu at (290.0, 48.0)
- added R3: 4.7k, Resistor_SMD:R_0805_2012Metric, F.Cu at (300.0, 48.0)
- added R4: 10k, Resistor_SMD:R_0805_2012Metric, F.Cu at (-14.9, -0.47)
- added SW66: RotaryEncoder_Switch, Rotary_Encoder:RotaryEncoder_Alps_EC11E-Switch_Vertical_H20mm, F.Cu at (-35.7, -2.87)
Routing:
- net GND: track 0.00 -> 480.6 mm
- net +3.3V: track 0.00 -> 426.7 mm, vias 0 -> 2
- net ENC_A: track 0.00 -> 378.4 mm, vias 0 -> 2
- net ENC_B: track 0.00 -> 365.1 mm, vias 0 -> 1
- net ENC_SW: track 0.00 -> 351.7 mm, vias 0 -> 1
- net COL0: track 96.3 -> 396.5 mm, vias 0 -> 1
- net COL1: track 97.4 -> 376.3 mm, vias 0 -> 1
- net COL14: track 358.1 -> 116.8 mm
- net COL2: track 126.5 -> 363.5 mm
- net COL3: track 125.2 -> 318.7 mm
- net COL13: track 296.5 -> 111.2 mm
- net COL4: track 160.0 -> 323.1 mm
- net COL12: track 311.9 -> 172.4 mm
- net COL5: track 152.5 -> 279.2 mm
- net COL11: track 293.2 -> 204.0 mm
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Other:
- board size 319.8 x 101.2 mm -> 345.1 x 101.2 mm

Commit message: new firmware and case
Parts:
- removed H7, H8: MountingHole_2.7mm_M2.5_Clean, Winter60_Mounting:MountingHole_2.7mm_M2.5_Clean
- added H10: MountingHole_2.7mm_M2.5_Clean, Winter60_Mounting:MountingHole_2.7mm_M2.5_Clean, F.Cu at (281.0, 28.6)
- added H11: MountingHole_2.7mm_M2.5_Clean, Winter60_Mounting:MountingHole_2.7mm_M2.5_Clean, F.Cu at (281.0, 66.7)
- added REF**: MountingHole_2.5mm, MountingHole:MountingHole_2.5mm, F.Cu at (286.7, 61.9)
- added REF1: MountingHole_2.5mm, MountingHole:MountingHole_2.5mm, F.Cu at (308.6, 61.9)
- moved J1 15.4 mm to (301.7, 85.0), turned to -90 degrees
- moved A1 7.20 mm to (297.2, 14.0)
- moved R1 7.20 mm to (287.2, 48.0)
- moved R2 7.20 mm to (297.2, 48.0)
- moved R3 7.20 mm to (307.2, 48.0)
Routing:
- net +3.3V: track 426.7 -> 497.0 mm, vias 2 -> 1
- net ROW4: track 424.7 -> 378.6 mm, vias 8 -> 5
- net ROW3: track 427.0 -> 397.0 mm, vias 11 -> 10
- net ROW0: track 377.3 -> 404.1 mm
- net COL9: track 213.8 -> 238.3 mm
- net ENC_B: track 365.1 -> 388.3 mm, vias 1 -> 2
- net SCL: track 55.5 -> 76.7 mm
- net SDA: track 54.5 -> 74.5 mm
- net COL5: track 279.2 -> 293.3 mm
- net COL3: track 318.7 -> 332.6 mm, vias 1 -> 2
- net ENC_A: track 378.4 -> 392.1 mm, vias 2 -> 1
- net COL13: track 111.2 -> 123.5 mm
- net COL12: track 172.4 -> 184.7 mm
- net GND: track 480.6 -> 491.8 mm
- net COL7: track 268.4 -> 279.1 mm
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Other:
- board size 345.1 x 101.2 mm -> 352.1 x 101.2 mm
