File: PCB/winter.kicad_pcb (KiCad board)
At the start: 2 copper layers, 352.1 x 101.2 mm, 152 parts, among them J1 Conn_01x04, SW1 SW_Push, SW10 SW_Push, SW11 SW_Push, SW12 SW_Push, SW13 SW_Push, SW14 SW_Push, SW15 SW_Push, SW16 SW_Push, SW17 SW_Push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

Commit message: new branding and silkscreen
Parts:
- added G***: LOGO, LOGO, F.Cu at (135.3, 37.9)
